File: eagle files/Safety Valve SMT.brd (EAGLE design)
At the start: 39.4 x 107.9 mm, 31 parts, among them IC1 TL072

Commit message: re-arranged the traces a bit
Routing:
- net N$7: track 47.0 -> 43.2 mm
- net GND: track 237.0 -> 240.1 mm
- net N$20: track 31.8 -> 29.3 mm
- net N$12: track 37.4 -> 39.3 mm
- net N$14: track 83.0 -> 81.4 mm
- net N$17: track 50.4 -> 49.2 mm
- net +12V: track 172.4 -> 173.5 mm

Commit message: Tidied up a bit
- Mittered traces
- Enlarged the width of them
- fixed two overlapping
Routing:
- net N$19: track 27.3 -> 123.7 mm, vias 0 -> 1
- net N$23: track 50.6 -> 42.8 mm
- net N$1: track 88.4 -> 82.5 mm
- net GND: track 240.1 -> 245.4 mm
- net N$17: track 49.2 -> 44.4 mm
- net -12V: track 107.2 -> 102.5 mm
- net +12V: track 173.5 -> 169.3 mm
- net N$4: track 80.9 -> 77.2 mm
- net N$22: track 33.1 -> 30.6 mm
- net N$7: track 43.2 -> 41.2 mm
- net N$21: track 42.5 -> 41.1 mm
- net N$5: track 38.4 -> 37.7 mm

Commit message: Added CV IN
Parts:
- removed GAIN-IN, TONE-IN: SOCKET_MONO_3.5MMPJ301M-12, GMSN:PJ301M-12
- added GAIN_IN, TONE_IN: THONKICONNNEW, MusicThingModular:WQP-PJ301M-12_JACK
- added R12, R15: 39k, GMSN:R0805
- added R13, R2: value, GMSN:R0805
- added R14, R7: 10k, GMSN:R0805
- added T1, T2: (no value), MusicThingModular:SOT23-BEC
- added U1, U2: TL072_SMD, MusicThingModular:SO08
- GAIN, TONE: value 100k -> (none); device GMSN:POTENTIOMETER_9MM -> MusicThingModular:9MM_SNAP-IN_POT
- moved LDR2 196.1 mm to (-6.35, -135.9), turned to 0 degrees
- moved TONE 155.9 mm to (-15.2, -110.5)
- moved GAIN 106.3 mm to (2.54, -59.7)
- moved C1 3.56 mm to (12.7, 78.9)
- moved R11 3.17 mm to (12.7, 75.6)
Connections:
- new net N$24: R12.1, R2.1, R7.1, U1.3
- new net N$25: GAIN.2, R2.2
- new net N$26: GAIN_IN.P$1_TIP, R7.2
- new net N$27: LDR1.2, T1.C
- new net N$28: R13.1, R14.1, R15.1, U2.3
- new net N$29: R13.2, TONE.2
- new net N$30: R14.2, TONE_IN.P$1_TIP
- new net N$31: LDR2.2, T2.C
- new net V+: U1.8, U2.8
- new net V-: U1.4, U2.4
- net +12V: now also GAIN.3, TONE.3
- net -12V: now also GAIN.1, LDR1.1, LDR2.1, TONE.1
- net GND: now also R12.2, R15.2; no longer GAIN.P$1, LDR1.4, LDR2.4, TONE.P$1, TONE.P$2
- net N$1: now also T2.E, U2.2; no longer GAIN.P$2, GAIN.P$3, LDR1.3, V1.P$3
- net N$17: now also T2.B, U2.1; no longer C7.2, LDR2.3, TONE.P$3
- net N$20: now also LDR1.3, V1.P$3; no longer LDR2.2, TONE-IN.TIP
- net N$21: now also C7.2, LDR2.3; no longer LDR2.1, TONE-IN.GND
- net N$22: now also T1.E, U1.2; no longer GAIN-IN.TIP, LDR1.2
- net N$23: now also T1.B, U1.1; no longer GAIN-IN.GND, LDR1.1
Routing:
- net N$1: track 82.5 -> 0.00 mm
- net GND: track 245.4 -> 191.5 mm
- net N$17: track 44.4 -> 0.00 mm
- net N$23: track 42.8 -> 0.00 mm
- net N$21: track 41.1 -> 0.00 mm
- net N$22: track 30.6 -> 0.00 mm
- net N$20: track 29.3 -> 0.00 mm
- net N$18: track 14.2 -> 9.70 mm
- net N$7: track 41.2 -> 44.3 mm

Commit message: added a missing resistor
Parts:
- added R16, R17: 470, GMSN:M0805
Connections:
- net +12V: now also R16.1, R17.1
- net N$1: now also R17.2
- net N$22: now also R16.2
Changed lines of the file:
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@@
 </element>
 <element name="TONE_IN" library="MusicThingModular" package="WQP-PJ301M-12_JACK" value="THONKICONNNEW" x="-27.94" y="-139.7"/>
+<element name="R16" library="GMSN" package="M0805" value="470" x="-33.02" y="-172.72">
+<attribute name="SPICEPREFIX" value="R" x="-33.02" y="-172.72" size="1.778" layer="27" display="off"/>
+</element>
+<element name="R17" library="GMSN" package="M0805" value="470" x="-33.02" y="-179.07">
+<attribute name="SPICEPREFIX" value="R" x="-33.02" y="-179.07" size="1.778" layer="27" display="off"/>
+</element>
 </elements>
 <signals>
@@
 <contactref element="GAIN" pad="3"/>
 <contactref element="TONE" pad="3"/>
+<contactref element="R16" pad="1"/>
+<contactref element="R17" pad="1"/>
+<wire x1="-33.97" y1="-172.72" x2="-33.97" y2="-179.07" width="0" layer="19" extent="1-1"/>
+<wire x1="-12.74" y1="-117.49" x2="-33.97" y2="-172.72" width="0" layer="19" extent="1-1"/>
 <wire x1="5.04" y1="-66.69" x2="-12.74" y2="-117.49" width="0" layer="19" extent="1-1"/>
 <wire x1="3.81" y1="1.27" x2="5.04" y2="-66.69" width="0" layer="19" extent="16-16"/>
@@
 <contactref element="T1" pad="E"/>
 <contactref element="U1" pad="2"/>
+<contactref element="R16" pad="2"/>
+<wire x1="-14.29" y1="-9.99" x2="-32.07" y2="-172.72" width="0" layer="19" extent="1-1"/>
 <wire x1="-14.605" y1="-1.33" x2="-14.29" y2="-9.99" width="0" layer="19" extent="1-1"/>
 </signal>
@@
 <contactref element="T2" pad="E"/>
 <contactref element="U2" pad="2"/>
+<contactref element="R17" pad="2"/>
+<wire x1="-31.115" y1="-166.43" x2="-32.07" y2="-179.07" width="0" layer="19" extent="1-1"/>
 <wire x1="-21.91" y1="-159.85" x2="-31.115" y2="-166.43" width="0" layer="19" extent="1-1"/>
 </signal>

Commit message: grounded the jacks in
Connections:
- net GND: now also GAIN_IN.P$3_SLEEVE, TONE_IN.P$3_SLEEVE
Changed lines of the file:
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@@
 <contactref element="R12" pad="2"/>
 <contactref element="R15" pad="2"/>
-<wire x1="-14.29" y1="-91.44" x2="-5.4" y2="-158.75" width="0" layer="19" extent="1-1"/>
-<wire x1="10.16" y1="3.66" x2="-14.29" y2="-91.44" width="0" layer="19" extent="1-1"/>
+<contactref element="GAIN_IN" pad="P$3_SLEEVE"/>
+<contactref element="TONE_IN" pad="P$3_SLEEVE"/>
+<wire x1="-5.4" y1="-158.75" x2="-27.94" y2="-146.2" width="0" layer="19" extent="1-1"/>
+<wire x1="-14.29" y1="-91.44" x2="-27.94" y2="-146.2" width="0" layer="19" extent="1-1"/>
+<wire x1="-27.94" y1="-85.24" x2="-14.29" y2="-91.44" width="0" layer="19" extent="1-1"/>
+<wire x1="10.16" y1="3.66" x2="-27.94" y2="-85.24" width="0" layer="19" extent="1-1"/>
 <wire x1="11.43" y1="43.18" x2="26.71" y2="27.07440625" width="0" layer="19" extent="16-16"/>
 </signal>
