File: eagle files/Safety Valve SMT.sch (EAGLE design)
At the start: 31 parts, among them IC1 TL072

Commit message: Added CV IN
Parts:
- removed GAIN-IN, TONE-IN: SOCKET_MONO_3.5MMPJ301M-12, GMSN:SOCKET_MONO_3.5MMPJ301M-12
- added GAIN_IN, TONE_IN: THONKICONNNEW, MusicThingModular:THONKICONNNEW
- added R12, R15: 39k, GMSN:RESISTOR_USR0805
- added R13, R2: value, GMSN:RESISTOR_USR0805
- added R14, R7: 10k, GMSN:RESISTOR_USR0805
- added T1, T2: (no value), MusicThingModular:BC807-16-PNP-SOT23-BEC
- added U1, U2: TL072_SMD, MusicThingModular:TL072_SMD
- GAIN, TONE: value 100k -> (none); device GMSN:RESISTOR_VARIABLE9MM_POT -> MusicThingModular:9MM_SNAP-IN_POT_; SPICEPREFIX X -> (none)
Connections:
- new net N$24: R12.1, R2.1, R7.1, U1A.+IN
- new net N$25: GAIN.S, R2.2
- new net N$26: GAIN_IN.TIP, R7.2
- new net N$27: LDR1.LED+, T1.C
- new net N$28: R13.1, R14.1, R15.1, U2A.+IN
- new net N$29: R13.2, TONE.S
- new net N$30: R14.2, TONE_IN.TIP
- new net N$31: LDR2.LED+, T2.C
- net +12V: now also GAIN.E, TONE.E
- net -12V: now also GAIN.A, LDR1.LED-, LDR2.LED-, TONE.A
- net GND: now also R12.2, R15.2; no longer GAIN.1, LDR1.RES2, LDR2.RES2, TONE.1, TONE.2
- net N$1: now also T2.E, U2A.-IN; no longer GAIN.2, GAIN.3, LDR1.RES1, V1A.TK
- net N$17: now also T2.B, U2A.OUT; no longer C7.2, LDR2.RES1, TONE.3
- net N$20: now also LDR1.RES1, V1A.TK; no longer LDR2.LED+, TONE-IN.TIP
- net N$21: now also C7.2, LDR2.RES1; no longer LDR2.LED-, TONE-IN.SLEEVE
- net N$22: now also T1.E, U1A.-IN; no longer GAIN-IN.TIP, LDR1.LED+
- net N$23: now also T1.B, U1A.OUT; no longer GAIN-IN.SLEEVE, LDR1.LED-
Other:
- moved on the sheet: LDR1, LDR2

Commit message: added a missing resistor
Parts:
- added R16, R17: 470, GMSN:RESISTOR_USM0805
Connections:
- net +12V: now also R16.1, R17.1
- net N$1: now also R17.2
- net N$22: now also R16.2
Changed lines of the file:
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@@
 <part name="SUPPLY7" library="supply2" library_urn="urn:adsk.eagle:library:372" deviceset="-12V" device=""/>
 <part name="SUPPLY8" library="supply2" library_urn="urn:adsk.eagle:library:372" deviceset="-12V" device=""/>
+<part name="R16" library="GMSN" deviceset="RESISTOR_US" device="M0805" value="470">
+<spice>
+<pinmapping spiceprefix="R">
+<pinmap gate="G$1" pin="1" pinorder="1"/>
+<pinmap gate="G$1" pin="2" pinorder="2"/>
+</pinmapping>
+</spice>
+<attribute name="SPICEPREFIX" value="R"/>
+</part>
+<part name="SUPPLY9" library="supply2" library_urn="urn:adsk.eagle:library:372" deviceset="+12V" device=""/>
+<part name="R17" library="GMSN" deviceset="RESISTOR_US" device="M0805" value="470">
+<spice>
+<pinmapping spiceprefix="R">
+<pinmap gate="G$1" pin="1" pinorder="1"/>
+<pinmap gate="G$1" pin="2" pinorder="2"/>
+</pinmapping>
+</spice>
+<attribute name="SPICEPREFIX" value="R"/>
+</part>
+<part name="SUPPLY10" library="supply2" library_urn="urn:adsk.eagle:library:372" deviceset="+12V" device=""/>
 </parts>
 <sheets>
@@
 <instance part="SUPPLY7" gate="G$1" x="38.1" y="-109.22"/>
 <instance part="SUPPLY8" gate="G$1" x="101.6" y="-127"/>
+<instance part="R16" gate="G$1" x="33.02" y="-132.08" rot="R90"/>
+<instance part="SUPPLY9" gate="+12V" x="25.4" y="-134.62"/>
+<instance part="R17" gate="G$1" x="96.52" y="-149.86" rot="R90"/>
+<instance part="SUPPLY10" gate="+12V" x="88.9" y="-152.4"/>
 </instances>
 <busses>
@@
 <pinref part="TONE" gate="G$1" pin="E"/>
 </segment>
+<segment>
+<pinref part="R16" gate="G$1" pin="1"/>
+<pinref part="SUPPLY9" gate="+12V" pin="+12V"/>
+<wire x1="33.02" y1="-137.16" x2="25.4" y2="-137.16" width="0.1524" layer="91"/>
+</segment>
+<segment>
+<pinref part="R17" gate="G$1" pin="1"/>
+<pinref part="SUPPLY10" gate="+12V" pin="+12V"/>
+<wire x1="96.52" y1="-154.94" x2="88.9" y2="-154.94" width="0.1524" layer="91"/>
+</segment>
 </net>
 <net name="N$5" class="0">
@@
 <pinref part="U1" gate="A" pin="-IN"/>
 <wire x1="7.62" y1="-116.84" x2="10.16" y2="-116.84" width="0.1524" layer="91"/>
+<pinref part="R16" gate="G$1" pin="2"/>
+<wire x1="33.02" y1="-124.46" x2="33.02" y2="-127" width="0.1524" layer="91"/>
+<junction x="33.02" y="-124.46"/>
 </segment>
 </net>
@@
 <pinref part="U2" gate="A" pin="-IN"/>
 <wire x1="71.12" y1="-134.62" x2="73.66" y2="-134.62" width="0.1524" layer="91"/>
-</segment>
-</net>
+<pinref part="R17" gate="G$1" pin="2"/>
+<wire x1="96.52" y1="-142.24" x2="96.52" y2="-144.78" width="0.1524" layer="91"/>
+<junction x="96.52" y="-142.24"/>
+</segment>
+</net>

Commit message: grounded the jacks in
Connections:
- net GND: now also GAIN_IN.SLEEVE, TONE_IN.SLEEVE
Other:
- moved on the sheet: GAIN_IN, TONE_IN
Changed lines of the file:
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@@
 </part>
 <part name="SUPPLY10" library="supply2" library_urn="urn:adsk.eagle:library:372" deviceset="+12V" device=""/>
+<part name="SUPPLY11" library="supply2" library_urn="urn:adsk.eagle:library:372" deviceset="GND" device=""/>
+<part name="SUPPLY12" library="supply2" library_urn="urn:adsk.eagle:library:372" deviceset="GND" device=""/>
 </parts>
 <sheets>
@@
 <instance part="R7" gate="G$1" x="-2.54" y="-144.78" rot="R180"/>
 <instance part="R12" gate="G$1" x="5.08" y="-157.48" rot="R270"/>
-<instance part="GAIN_IN" gate="G$1" x="-17.78" y="-142.24" rot="R180"/>
+<instance part="GAIN_IN" gate="G$1" x="-15.24" y="-147.32" rot="MR0"/>
 <instance part="LDR2" gate="G$1" x="99.06" y="-111.76" rot="R90"/>
 <instance part="SUPPLY4" gate="+12V" x="53.34" y="-119.38"/>
@@
 <instance part="R14" gate="G$1" x="60.96" y="-162.56" rot="R180"/>
 <instance part="R15" gate="G$1" x="68.58" y="-175.26" rot="R270"/>
-<instance part="TONE_IN" gate="G$1" x="45.72" y="-160.02" rot="R180"/>
+<instance part="TONE_IN" gate="G$1" x="48.26" y="-165.1" rot="MR0"/>
 <instance part="SUPPLY7" gate="G$1" x="38.1" y="-109.22"/>
 <instance part="SUPPLY8" gate="G$1" x="101.6" y="-127"/>
@@
 <instance part="R17" gate="G$1" x="96.52" y="-149.86" rot="R90"/>
 <instance part="SUPPLY10" gate="+12V" x="88.9" y="-152.4"/>
+<instance part="SUPPLY11" gate="GND" x="-10.16" y="-157.48"/>
+<instance part="SUPPLY12" gate="GND" x="53.34" y="-175.26"/>
 </instances>
 <busses>
@@
 <pinref part="R15" gate="G$1" pin="2"/>
 <pinref part="SUPPLY6" gate="GND" pin="GND"/>
+</segment>
+<segment>
+<pinref part="GAIN_IN" gate="G$1" pin="SLEEVE"/>
+<pinref part="SUPPLY11" gate="GND" pin="GND"/>
+<wire x1="-10.16" y1="-149.86" x2="-10.16" y2="-154.94" width="0.1524" layer="91"/>
+</segment>
+<segment>
+<pinref part="TONE_IN" gate="G$1" pin="SLEEVE"/>
+<pinref part="SUPPLY12" gate="GND" pin="GND"/>
+<wire x1="53.34" y1="-167.64" x2="53.34" y2="-172.72" width="0.1524" layer="91"/>
 </segment>
 </net>
@@
 <pinref part="GAIN_IN" gate="G$1" pin="TIP"/>
 <pinref part="R7" gate="G$1" pin="2"/>
-<wire x1="-12.7" y1="-144.78" x2="-7.62" y2="-144.78" width="0.1524" layer="91"/>
+<wire x1="-10.16" y1="-144.78" x2="-7.62" y2="-144.78" width="0.1524" layer="91"/>
 </segment>
 </net>
@@
 <pinref part="TONE_IN" gate="G$1" pin="TIP"/>
 <pinref part="R14" gate="G$1" pin="2"/>
-<wire x1="50.8" y1="-162.56" x2="55.88" y2="-162.56" width="0.1524" layer="91"/>
-</segment>
-</net>
+<wire x1="53.34" y1="-162.56" x2="55.88" y2="-162.56" width="0.1524" layer="91"/>
+</segment>
+</net>
